File: hardware/brainboardv1/brainboardv1.kicad_pcb (KiCad board)
At the start: 4 copper layers, 86.4 x 54.6 mm, 117 parts, among them P1 WP, P10 CONN_2X2, P2 CONN_14, P3 CONN_5X2, P4 BTRST, P5 GND, P6 -3V3, P7 3V3, P8 +2V5, P9 -2V5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

Commit message: More battery changes
Added power-down logic to battery board (currently faulty, need
revision); added fuel gauge, 2-pin JST, and BBB battery connector to
Brainboard R1.
TODO: Fix power-down logic (suggest dedicated power-button supervisor
like STM660x), add isolation so board can be safely plugged in to charge
Parts:
- added C57: 0.01uF, SM0603, F.Cu at (157.7, 132.7)
- added C58: 1uF, SM0603, F.Cu at (157.7, 134.8)
- added P11: JST, s2b-ph-sm4-tb, F.Cu at (118.1, 133.3)
- added P12: CONN_4, PIN_ARRAY_2X2, F.Cu at (139.8, 135.5)
- added P13: VBAT, PINTST, F.Cu at (151.4, 135.6)
- added P14: ~ALRT, PINTST, F.Cu at (151.3, 139.5)
- added R27: 180, SM0603, F.Cu at (151.3, 130.4)
- added R28: 1k, SM0603, F.Cu at (154.4, 130.5)
- added TH1: 10k NTC, SM0603, F.Cu at (157.8, 130.6)
- added U14: MAX17043, tdfn8, F.Cu at (147.1, 131.3)
- D2: value CONN -> CONNECT
- R10: value 10K -> 75k
Connections:
- R10 pad 1: +3.3V -> /BrainBoard Power/TS
- R10 pad 2: /BrainBoard AFE//RESET -> AGND
Routing:
- net /BrainBoard Power/TS: track 0.00 -> 2.51 mm
- net +3.3V: track 225.9 -> 223.4 mm
