File: hardware/brainboardv1/brainboardv1_afe.sch (KiCad schematic (older format))
At the start: 25 parts

Commit message: Nearly finished v1 sch & brd, await final check
Fixed errors from Rev 0, added MPU-6050 accelerometer/gyro for head
motion tracking, switched to +/-2.5V analog supply, added 2 bipolar
analog inputs for EOG tracking, added daisy-chain capability
Parts:
- removed R? (x2): 10K, ~, symbol R
- removed SJ?: SOLDERJUMPER_2WAYPASTE2&3, SparkFun-Passives-SJ_3_PASTE2&3, symbol SOLDERJUMPER_2WAYPASTE2&3
- added C50: 0.1uF, ~, symbol C
- added P10: CONN_2X2, ~, symbol CONN_2X2
- added R7: 10K, ~, symbol R
- added SJ2, SJ7: DAISY_CS, SparkFun-Passives-SJ_3_PASTE2&3, symbol SOLDERJUMPER_2WAYPASTE2&3
- added SJ6: DAISY_OUT, SparkFun-Passives-SJ_3_PASTE2&3, symbol SOLDERJUMPER_2WAYPASTE2&3
- added SJ8: CLKSEL, SparkFun-Passives-SJ_3_PASTE1&2, symbol SOLDERJUMPER_2WAYPASTE2&3
- SJ1: renamed from SJ?; value SOLDERJUMPER_2WAYPASTE2&3 -> REF-SRB2
- SJ3: renamed from SJ?; value SOLDERJUMPERNO -> NO BIAS FILT
- gave numbers to parts that had none: 20
Connections:
- net labels added: +2.5V, -2.5V, /CS_DAISY, /CS_MAIN, CLK, CLKSEL, DAISY, DAISY_IN, DAISY_OUT, DOUT
- net labels removed: +5VA, /RESET, 3V3, AIN3N, AIN4N, AIN5N, AIN6N, AIN7N, AIN8N, START
- wire segments 117 -> 137
- no-connect marks 6 -> 4
Other:
- note added: "For daisy-chain operation, use the following jumper settings:\nSJ2, SJ6, SJ7, SJ8 @ 2-3 for master AFE (provides clock and bias supply);\nSJ2, SJ6, SJ7, SJ8 @ 1-2 for additional AFEs"
- moved on the sheet: C10, C11, C12, C13, C14, C15, C16, C9, SJ3
