File: hardware/brainboard/brainboard_batteryv0/brainboard_batteryv0.sch (KiCad schematic (older format))
At the start: 64 parts, among them CON1 USB-MINI-B, P1 JST, P10 3V3, P2 VBAT, P3 GND, P4 BBB_PMIC, P5 ~ALRT, P6 VBUS, P7 WP, P8 EN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

Commit message: Thesis version
Finally able to commit again (Windows XP issues fixed by OS upgrade).
Added latest version of wearable BB, along with prototype "muscleboard"
2-channel board for EMG/ECG applications
Parts:
- removed P5: ~ALRT, ~, symbol TST
- removed Q1: SI2312, ~, symbol MOS_N_E
- added D6: ALRT, ~, symbol LED
- added R19: 2.2k, ~, symbol R
Connections:
- wire segments 329 -> 245
Other:
- note removed: "Reverse\npolarity\nprotection"
