File: hardware/brainboard/brainboardv1/brainboardv1.kicad_pcb (KiCad board)
At the start: 4 copper layers, 86.4 x 54.6 mm, 127 parts, among them P1 WP, P10 CONN_2X2, P11 JST, P12 CONN_4, P13 VBAT, P14 ~ALRT, P2 CONN_14, P3 CONN_5X2, P4 BTRST, P5 GND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

Commit message: Thesis version
Finally able to commit again (Windows XP issues fixed by OS upgrade).
Added latest version of wearable BB, along with prototype "muscleboard"
2-channel board for EMG/ECG applications
Parts:
- removed C57: 0.01uF, SM0603
- removed C58: 1uF, SM0603
- removed P11: JST, s2b-ph-sm4-tb
- removed P12: CONN_4, PIN_ARRAY_2X2
- removed P13: VBAT, PINTST
- removed P14: ~ALRT, PINTST
- removed R10: 75k, SM0603
- removed R27: 180, SM0603
- removed R28: 1k, SM0603
- removed TH1: 10k NTC, SM0603
- removed U14: MAX17043, tdfn8
- U3: footprint MSOP_8 -> msoic-8
- moved S2 20.3 mm to (146.7, 156.4), turned to 270 degrees
Connections:
- C2 pad 2: /BrainBoard AFE/BIASOUT -> BIAS
- R9 pad 1: /BrainBoard AFE/BIASOUT -> BIAS
- SJ3 pad 2: /BrainBoard AFE/BIASOUT -> BIAS
- U4 pad 63: /BrainBoard AFE/BIASOUT -> BIAS
Routing:
- net N-0000026: track 9.12 -> 33.1 mm
- net I2C2_SCL: track 59.1 -> 82.0 mm
- net I2C2_SDA: track 59.4 -> 73.0 mm
- net +3.3V: track 220.9 -> 232.5 mm
- net BIAS: track 21.6 -> 31.3 mm, vias 0 -> 1
- net /BrainBoard AFE/BIASOUT: track 9.14 -> 0.00 mm, vias 1 -> 0
- net AGND: track 498.8 -> 500.8 mm
