File: hardware/brainboard/brainboardv1/brainboardv1_bt.sch (KiCad schematic (older format))
At the start: 7 parts, among them P4 BTRST, U9 BLUETOOTH-RN42

Commit message: Thesis version
Finally able to commit again (Windows XP issues fixed by OS upgrade).
Added latest version of wearable BB, along with prototype "muscleboard"
2-channel board for EMG/ECG applications
Parts:
- D2: value CONNECT -> CONN
Changed lines of the file:
@@
 Sheet 4 7
 Title "BrainBoard: Open-Source Hardware for Wearable BCI"
-Date "23 jan 2014"
+Date "19 jun 2014"
 Rev "0"
 Comp "Virginia Commonwealth University"
@@
 P 7200 3800
 F 0 "D2" H 7200 3900 50  0000 C CNN
-F 1 "CONNECT" H 7200 3700 50  0000 C CNN
+F 1 "CONN" H 7200 3700 50  0000 C CNN
 F 2 "~" H 7200 3800 60  0000 C CNN
 F 3 "~" H 7200 3800 60  0000 C CNN
