File: hardware/muscleboard/muscleboardv0.sch (KiCad schematic (older format))
At the start: 33 parts, among them P1 BATT, P2 USB, P3 ICSP, U1 ATMEGA328P, U2 MCP73831T-DFN, U3 TPS73233, U4 BLUETOOTH-RN42, Y1 RESONATOR

Commit message: Fixed CLKSEL and START no-connects on muscleboard
Also removed extraneous components including battery voltage
divider--going to use ATMEGA328p's internal voltage reference to measure
AVCC instead. AVCC is now directly tied to VCC
Parts:
- removed C1, C3, C9: 0.1uF, ~, symbol C
- removed C12: 2.2uF, ~, symbol C
- removed L1: 10uH, ~, symbol INDUCTOR
- removed R1: 2.2M, ~, symbol R
- removed R2: 1M, ~, symbol R
Connections:
- net labels removed: AVCC, BATT_MON
- wire segments 144 -> 130
- no-connect marks 33 -> 34
Other:
- note removed: "Divider reduces 3.52V to 1.1V\nto trigger comparator with MCU's\non-chip bandgap reference"
- moved on the sheet: C11
Changed lines of the file:
@@
 Sheet 1 2
 Title ""
-Date "9 sep 2014"
+Date "21 oct 2014"
 Rev ""
 Comp ""
@@
 3.3V regulation
 $Comp
-L C C9
-U 1 1 53ADA71B
-P 3900 1600
-F 0 "C9" H 3900 1700 40  0000 L CNN
-F 1 "0.1uF" H 3906 1515 40  0000 L CNN
-F 2 "~" H 3938 1450 30  0000 C CNN
-F 3 "~" H 3900 1600 60  0000 C CNN
-	1    3900 1600
-	1    0    0    -1
-$EndComp
-$Comp
 L TPS732XX U3
 U 1 1 53ADA71C
@@
 $EndComp
 $Comp
-L C C12
-U 1 1 53ADA71E
-P 6750 1550
-F 0 "C12" H 6750 1650 40  0000 L CNN
-F 1 "2.2uF" H 6756 1465 40  0000 L CNN
-F 2 "~" H 6788 1400 30  0000 C CNN
-F 3 "~" H 6750 1550 60  0000 C CNN
-	1    6750 1550
-	1    0    0    -1
-$EndComp
-$Comp
 L C C11
 U 1 1 53ADA71F
-P 6450 1550
-F 0 "C11" H 6450 1650 40  0000 L CNN
-F 1 "10uF" H 6456 1465 40  0000 L CNN
-F 2 "~" H 6488 1400 30  0000 C CNN
-F 3 "~" H 6450 1550 60  0000 C CNN
-	1    6450 1550
+P 6600 1550
+F 0 "C11" H 6600 1650 40  0000 L CNN
+F 1 "10uF" H 6606 1465 40  0000 L CNN
+F 2 "~" H 6638 1400 30  0000 C CNN
+F 3 "~" H 6600 1550 60  0000 C CNN
+	1    6600 1550
 	1    0    0    -1
 $EndComp
@@
 	1    0    0    -1
 $EndComp
-$Comp
-L C C1
-U 1 1 53ACD26E
-P 1200 5600
-F 0 "C1" H 1200 5700 40  0000 L CNN
-F 1 "0.1uF" H 1206 5515 40  0000 L CNN
-F 2 "~" H 1238 5450 30  0000 C CNN
-F 3 "~" H 1200 5600 60  0000 C CNN
-F 4 "Digikey" H 1200 5600 60  0001 C CNN "Distributor"
-F 5 "1276-1443-1-ND" H 1200 5600 60  0001 C CNN "PN"
-	1    1200 5600
-	1    0    0    -1
-$EndComp
-$Comp
-L GND #PWR021
-U 1 1 53ACD26F
-P 1200 5850
-F 0 "#PWR021" H 1200 5850 30  0001 C CNN
-F 1 "GND" H 1200 5780 30  0001 C CNN
-F 2 "~" H 1200 5850 60  0000 C CNN
-F 3 "~" H 1200 5850 60  0000 C CNN
-	1    1200 5850
-	1    0    0    -1
-$EndComp
-$Comp
-L INDUCTOR L1
-U 1 1 53ACD270
-P 2000 4900
-F 0 "L1" V 2100 4900 40  0000 C CNN
-F 1 "10uH" V 1950 4900 40  0000 C CNN
-F 2 "~" H 2000 4900 60  0000 C CNN
-F 3 "~" H 2000 4900 60  0000 C CNN
-F 4 "Digikey" V 2000 4900 60  0001 C CNN "Distributor"
-F 5 "445-3166-1-ND" V 2000 4900 60  0001 C CNN "PN"
-	1    2000 4900
-	0    -1   -1   0
-$EndComp
 Text Label 4300 6100 0    51   ~ 0
 USER_LED
@@
 Text Label 4300 5900 0    51   ~ 0
 BT_CONN
-$Comp
-L R R1
-U 1 1 53ACD273
-P 1200 6450
-F 0 "R1" V 1280 6450 40  0000 C CNN
-F 1 "2.2M" V 1207 6451 40  0000 C CNN
-F 2 "~" V 1130 6450 30  0000 C CNN
-F 3 "~" H 1200 6450 30  0000 C CNN
-F 4 "Digikey" V 1200 6450 60  0001 C CNN "Distributor"
-F 5 "1276-4295-1-ND" V 1200 6450 60  0001 C CNN "PN"
-	1    1200 6450
-	1    0    0    -1
-$EndComp
-$Comp
-L R R2
-U 1 1 53ACD274
-P 1200 7050
-F 0 "R2" V 1280 7050 40  0000 C CNN
-F 1 "1M" V 1207 7051 40  0000 C CNN
-F 2 "~" V 1130 7050 30  0000 C CNN
-F 3 "~" H 1200 7050 30  0000 C CNN
-F 4 "Digikey" V 1200 7050 60  0001 C CNN "Distributor"
-F 5 "RMCF0402JT1M00CT-ND" V 1200 7050 60  0001 C CNN "PN"
-	1    1200 7050
-	1    0    0    -1
-$EndComp
-$Comp
-L GND #PWR022
-U 1 1 53ACD275
-P 1200 7450
-F 0 "#PWR022" H 1200 7450 30  0001 C CNN
-F 1 "GND" H 1200 7380 30  0001 C CNN
-F 2 "~" H 1200 7450 60  0000 C CNN
-F 3 "~" H 1200 7450 60  0000 C CNN
-	1    1200 7450
-	1    0    0    -1
-$EndComp
-Text Notes 1300 7450 0    51   ~ 0
-Divider reduces 3.52V to 1.1V\nto trigger comparator with MCU's\non-chip bandgap reference
-$Comp
-L +BATT #PWR023
-U 1 1 53ACD276
-P 1200 6150
-F 0 "#PWR023" H 1200 6100 20  0001 C CNN
-F 1 "+BATT" H 1200 6250 30  0000 C CNN
-F 2 "~" H 1200 6150 60  0000 C CNN
-F 3 "~" H 1200 6150 60  0000 C CNN
-	1    1200 6150
-	1    0    0    -1
-$EndComp
-Text Label 2050 6750 2    51   ~ 0
-BATT_MON
-Text Label 4700 6350 2    51   ~ 0
-BATT_MON
 NoConn ~ 8050 5450
 NoConn ~ 8050 5550
@@
 FACTORY_RESET
 $Comp
-L GND #PWR024
+L GND #PWR021
 U 1 1 53ACD277
 P 8100 6700
-F 0 "#PWR024" H 8100 6700 30  0001 C CNN
+F 0 "#PWR021" H 8100 6700 30  0001 C CNN
 F 1 "GND" H 8100 6630 30  0001 C CNN
 F 2 "~" H 8100 6700 60  0000 C CNN
@@
 	1    0    0    -1
 $EndComp
-$Comp
-L C C3
-U 1 1 53ACD281
-P 1600 7050
-F 0 "C3" H 1600 7150 40  0000 L CNN
-F 1 "0.1uF" H 1606 6965 40  0000 L CNN
-F 2 "~" H 1638 6900 30  0000 C CNN
-F 3 "~" H 1600 7050 60  0000 C CNN
-F 4 "Digikey" H 1600 7050 60  0001 C CNN "Distributor"
-F 5 "1276-1443-1-ND" H 1600 7050 60  0001 C CNN "PN"
-	1    1600 7050
-	1    0    0    -1
-$EndComp
-Text Label 2250 5250 0    51   ~ 0
-AVCC
 Text Label 2250 5350 0    51   ~ 0
 AREF
@@
 Text GLabel 1900 4650 0    51   Input ~ 0
 ~MCU_RESET
-$Comp
-L PWR_FLAG #FLG025
-U 1 1 53ACD285
-P 1200 4900
-F 0 "#FLG025" H 1200 4995 30  0001 C CNN
-F 1 "PWR_FLAG" H 1200 5080 30  0000 C CNN
-F 2 "~" H 1200 4900 60  0000 C CNN
-F 3 "~" H 1200 4900 60  0000 C CNN
-	1    1200 4900
-	1    0    0    -1
-$EndComp
 NoConn ~ 8050 5850
 NoConn ~ 8050 5650
@@
 MCU_RX
 $Comp
-L +3.3V #PWR026
+L +3.3V #PWR022
 U 1 1 53ADAB68
 P 2400 4000
-F 0 "#PWR026" H 2400 3960 30  0001 C CNN
+F 0 "#PWR022" H 2400 3960 30  0001 C CNN
 F 1 "+3.3V" H 2400 4110 30  0000 C CNN
 F 2 "~" H 2400 4000 60  0000 C CNN
@@
 $EndComp
 $Comp
-L +3.3V #PWR027
+L +3.3V #PWR023
 U 1 1 53ADAB6E
 P 6350 4350
-F 0 "#PWR027" H 6350 4310 30  0001 C CNN
+F 0 "#PWR023" H 6350 4310 30  0001 C CNN
 F 1 "+3.3V" H 6350 4460 30  0000 C CNN
 F 2 "~" H 6350 4350 60  0000 C CNN
@@
 NoConn ~ 4300 6650
 $Comp
-L GND #PWR028
+L GND #PWR024
 U 1 1 53ADBAD2
 P 6300 5750
-F 0 "#PWR028" H 6300 5750 30  0001 C CNN
+F 0 "#PWR024" H 6300 5750 30  0001 C CNN
 F 1 "GND" H 6300 5680 30  0001 C CNN
 F 2 "~" H 6300 5750 60  0000 C CNN
@@
 $EndComp
 $Comp
-L +3.3V #PWR029
+L +3.3V #PWR025
 U 1 1 53ADE4B6
 P 6850 2500
-F 0 "#PWR029" H 6850 2460 30  0001 C CNN
+F 0 "#PWR025" H 6850 2460 30  0001 C CNN
 F 1 "+3.3V" H 6850 2610 30  0000 C CNN
 F 2 "~" H 6850 2500 60  0000 C CNN
@@
 $EndComp
 $Comp
-L GND #PWR030
+L GND #PWR026
 U 1 1 53B3483A
 P 2000 5850
-F 0 "#PWR030" H 2000 5850 30  0001 C CNN
+F 0 "#PWR026" H 2000 5850 30  0001 C CNN
 F 1 "GND" H 2000 5780 30  0001 C CNN
 F 2 "~" H 2000 5850 60  0000 C CNN
@@
 Wire Wire Line
 	5450 5050 4300 5050
-Connection ~ 1200 4900
-Wire Wire Line
-	2400 4000 2400 5000
+Wire Wire Line
+	2400 4000 2400 5250
 Wire Wire Line
 	8100 6350 8100 6700
-Connection ~ 1200 7350
-Wire Wire Line
-	1600 7350 1600 7250
-Wire Wire Line
-	1200 7350 1600 7350
-Connection ~ 1600 6750
-Wire Wire Line
-	1600 6850 1600 6750
 Wire Wire Line
 	5800 4550 5800 5250
@@
 Wire Wire Line
 	5800 4550 6450 4550
-Connection ~ 1200 6750
-Wire Wire Line
-	1200 6700 1200 6800
-Wire Wire Line
-	1200 6750 2050 6750
-Wire Wire Line
-	1200 7300 1200 7450
-Wire Wire Line
-	1200 6150 1200 6200
 Wire Wire Line
 	5500 5450 5500 7050
@@
 Wire Wire Line
 	2000 4050 2000 4100
-Connection ~ 1200 5250
-Wire Wire Line
-	1200 4900 1700 4900
-Wire Wire Line
-	1200 4900 1200 5400
-Wire Wire Line
-	1200 5850 1200 5800
-Wire Wire Line
-	4300 6350 4700 6350
 Connection ~ 2250 4650
 Wire Wire Line
@@
 Connection ~ 2400 4900
 Wire Wire Line
-	2300 4900 2450 4900
-Wire Wire Line
 	2000 4500 2000 4550
 Wire Wire Line
@@
 Wire Wire Line
 	1900 4650 2450 4650
-Wire Wire Line
-	1200 5250 2450 5250
 Wire Wire Line
 	6000 2550 5950 2550
@@
 Wire Wire Line
 	3900 1850 4350 1850
-Wire Wire Line
-	3900 1800 3900 2000
 Connection ~ 4250 1200
 Wire Wire Line
@@
 	3450 1100 3450 1400
 Connection ~ 3450 1200
-Connection ~ 3900 1850
-Wire Wire Line
-	3900 1200 3900 1400
-Connection ~ 6600 1750
 Wire Wire Line
 	6600 1750 6600 2000
-Wire Wire Line
-	6450 1750 6750 1750
-Connection ~ 6600 1350
-Wire Wire Line
-	6450 1350 6750 1350
 Wire Wire Line
 	5300 1900 6000 1900
@@
 Wire Wire Line
 	5750 1200 6600 1200
-Connection ~ 3900 1200
 Connection ~ 5300 1900
 Wire Wire Line
@@
 	4250 3250 4450 3250
 Connection ~ 4450 3250
+Wire Wire Line
+	2450 4900 2400 4900
+Wire Wire Line
+	2400 5250 2450 5250
+Connection ~ 2400 5000
+Wire Wire Line
+	3900 1850 3900 2000
+NoConn ~ 4300 6350
 $EndSCHEMATC
