File: hardware/muscleboard/muscleboardv0_afe.sch (KiCad schematic (older format))
At the start: 21 parts, among them P4 ELEC, U5 ADS1291, U6 ADXL362

Commit message: Fixed CLKSEL and START no-connects on muscleboard
Also removed extraneous components including battery voltage
divider--going to use ATMEGA328p's internal voltage reference to measure
AVCC instead. AVCC is now directly tied to VCC
Parts:
- removed C15, C23, C25: 0.1uF, ~, symbol C
- added R11, R13, R14, R6: 10k, ~, symbol R
Connections:
- net +3.3V: now also U5.14 (CLKSEL)
- net GND: now also U5.16 (START)
- new net: R11.2, R13.2, R14.2, R6.2, U5.12 (AVDD)
- new net: R6.1, U5.31 (RESP_MODP)
- new net: R11.1, U5.32 (RESP_MODN)
- new net: R14.1, U5.5 (IN2N)
- new net: R13.1, U5.6 (IN2P)
- no-connect marks 7 -> 5
Other:
- moved on the sheet: C16, C22, C24
