File: hardware/muscleboard/muscleboardv1/muscleboardv1.sch (KiCad schematic (older format))
At the start: 29 parts, among them P1 BATT, P2 USB, P3 ICSP, U1 ATMEGA328P, U2 MCP73831T-DFN, U3 TPS73233, U4 BLUETOOTH-RN42, Y1 RESONATOR

Commit message: Fixed CLKSEL and START no-connects on muscleboard
Also removed extraneous components including battery voltage
divider--going to use ATMEGA328p's internal voltage reference to measure
AVCC instead. AVCC is now directly tied to VCC
Parts:
- removed C10: 0.01uF, ~, symbol C
- removed C11: 10uF, ~, symbol C
- removed C2, C3, C5: 0.1uF, ~, symbol C
- removed C4, C8: 4.7uF, ~, symbol C
- removed D1: CHG, ~, symbol LED
- removed D2: LSM115JE3/TR13, ~, symbol DIODESCH
- removed D3: RED, ~, symbol LED
- removed MTG1: MHOLE, symbol MHOLE
- removed P1: BATT, ~, symbol CONN_2
- removed P2: USB, ~, symbol USB-MINI-B
- removed P3: ICSP, ~, symbol CONN_3X2
- removed R1: 2.2M, ~, symbol R
- removed R2: 1M, ~, symbol R
- removed R3, R5: 10k, ~, symbol R
- removed R4, R7: 2.2k, ~, symbol R
- removed S2: CHG/ON, ~, symbol SPDT
- removed TP1: GND, ~, symbol TST
- removed TP3: FACT, ~, symbol TESTPOINT
- removed U3: TPS73233, ~, symbol TPS732XX
- removed U4: BLUETOOTH-RN42, ~, symbol BLUETOOTH-RN42
- added C? (x5): 0.1uF, ~, symbol C
- added C?: 0.01uF, ~, symbol C
- added C?: 2.2uF, ~, symbol C
- added C?: 10uF, ~, symbol C
- added C? (x2): 4.7uF, ~, symbol C
- added D?: CHG, ~, symbol LED
- added D?: LSM115JE3/TR13, ~, symbol DIODESCH
- added D?: RED, ~, symbol LED
- added L?: 10uH, ~, symbol INDUCTOR
- added MTG?: MHOLE, symbol MHOLE
- added P?: BATT, ~, symbol CONN_2
- added P?: USB, ~, symbol USB-MINI-B
- added P?: ICSP, ~, symbol CONN_3X2
- added R? (x2): 10k, ~, symbol R
- added R? (x2): 2.2k, ~, symbol R
- added R?: 2.2M, ~, symbol R
- added R?: 1M, ~, symbol R
- added S?: CHG/ON, ~, symbol SPDT
- added TP?: GND, ~, symbol TST
- added TP?: FACT, ~, symbol TESTPOINT
- added U?: TPS73233, ~, symbol TPS732XX
- added U?: BLUETOOTH-RN42, ~, symbol BLUETOOTH-RN42
Connections:
- net labels added: AVCC
- wire segments 138 -> 144
